Commit message: Add ball catching, kicking, and trajectory prediction system
- table_mover.py: ball catching with state machine (WAITING/CATCHING/CAUGHT/RETURNING),
  smooth accel/decel, collision detection via ball_position topic
- kick.py: twist-based kick motion (windup +Y then drive -Y) with ready state
- trajectory_predictor.py: ball arrival prediction at y=0.6 workspace boundary
- ball_tracker.py: improved tracking with smoothing and loss timeout
- BallArrival.msg: new message type for ball arrival predictions
- display_vertical.launch: custom zone filter with sleep-based kill of default filter
- goal_tracker.py, HSV_tuner.py: new utility scripts
- ball_game.launch: new launch file for full game setup
- Removed frame_calibration.py and ur5e_follower.py

Co-Authored-By: Claude Sonnet 4.6 <noreply@anthropic.com>

File: src/ur5e_scene/urdf/ur5e_table_vertical.urdf (robot description, URDF)
Before this commit: robot cu_ur5e, 24 links, 23 joints
Links:
- added link arm_ee_adapter; collision mesh filename=package://ur5e_scene/meshes/end_effector.stl scale=0.001 0.001 0.001; visual mesh filename=package://ur5e_scene/meshes/end_effector.stl scale=0.001 0.001 0.001
Joints:
- added joint arm_flange_to_adapter: type fixed, parent arm_tool0, child arm_ee_adapter, origin xyz=0 0 0.023 rpy=1.57 0 1.63
